File: pcb/pico2-vga-adapter/pico2-vga-adapter.kicad_pcb (KiCad board)
At the start: 2 copper layers, 70.1 x 48.3 mm, 69 parts, among them J1 USB_B_Micro, J2 VGA, J3 CONN, J4 SM03B-SRSS-TB, J6 UART, Q1 BSS138, Q10 BSS138, Q2 BSS138, Q3 BSS138, Q4 BSS138, Q5 BSS138, Q6 BSS138, Q7 BSS138, Q8 BSS138, Q9 BSS138, SW1 SW_Push, SW2 SW_Push, U1 RP2350_60QFN, U2 NCP1117-3.3_SOT223, U3 W25Q128JVS, Y1 ABM8-272-T3

Commit message: Routing
Parts:
- removed Q1, Q10, Q2, Q3, Q4, Q5, Q6, Q7, Q8, Q9: BSS138, Package_TO_SOT_SMD:SOT-23
- removed RN1, RN2, RN3, RN4, RN5: 10k, Resistor_SMD:R_Array_Convex_4x0603
- added U4: SN74CBTD3861PWR, Package_SO:TSSOP-24_4.4x7.8mm_P0.65mm, F.Cu at (126.5, 102.6)
- moved J3 28.7 mm to (142.5, 114.3), turned to -90 degrees
Routing:
- net GND: track 51.6 -> 143.8 mm, vias 27 -> 30
- net +5V: track 3.14 -> 90.8 mm, vias 0 -> 5
- net LD1: track 5.76 -> 85.2 mm, vias 1 -> 2
- net VSYNC: track 0.00 -> 74.7 mm, vias 0 -> 1
- net TX: track 0.00 -> 67.4 mm, vias 0 -> 1
- net LD4: track 6.03 -> 71.0 mm, vias 1 -> 2
- net LD3: track 6.05 -> 70.9 mm, vias 1 -> 2
- net HSYNC: track 0.00 -> 64.7 mm, vias 0 -> 1
- net LD2: track 5.90 -> 67.9 mm, vias 1 -> 2
- net LD7: track 6.46 -> 68.0 mm, vias 1 -> 4
- net LD0: track 5.65 -> 66.7 mm, vias 1 -> 4
- net LD6: track 6.32 -> 63.4 mm, vias 1 -> 4
- net LD5: track 6.17 -> 62.4 mm, vias 1 -> 2
- net COL_R1: track 0.00 -> 54.2 mm, vias 0 -> 2
- net L_LATCH: track 5.98 -> 56.5 mm, vias 1 -> 2
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- added copper zone on B.Cu, net GND

Commit message: Adding components
Parts:
- added BZ1: Buzzer, Buzzer_Beeper:Buzzer_15x7.5RM7.6, F.Cu at (137.9, 100.0)
Connections:
- U1 pad 34: /GPIO22 -> unconnected-(U1-GPIO22-Pad34)
- U1 pad 35: /GPIO23 -> unconnected-(U1-GPIO23-Pad35)
- U1 pad 36: /GPIO24 -> unconnected-(U1-GPIO24-Pad36)
- U1 pad 37: /GPIO25 -> unconnected-(U1-GPIO25-Pad37)
- U1 pad 40: /GPIO26_ADC0 -> unconnected-(U1-GPIO26_ADC0-Pad40)
- U1 pad 41: /GPIO27_ADC1 -> unconnected-(U1-GPIO27_ADC1-Pad41)
- U1 pad 42: /GPIO28_ADC2 -> unconnected-(U1-GPIO28_ADC2-Pad42)
- U1 pad 43: /GPIO29_ADC3 -> unconnected-(U1-GPIO29_ADC3-Pad43)
Routing:
- net AUDIO: track 6.21 -> 99.7 mm, vias 1 -> 2
- net GND: track 143.8 -> 140.7 mm, vias 30 -> 32
- net COL_B1: track 36.5 -> 38.5 mm
- net COL_R2: track 30.0 -> 30.9 mm
- net L_LATCH: track 56.5 -> 55.8 mm
- net COL_G0: track 30.0 -> 30.6 mm
- net COL_B0: track 35.8 -> 36.3 mm
- net COL_R0: track 49.7 -> 50.3 mm

Commit message: Finalizing adapter design
Parts:
- removed R13, R17: 150, Resistor_SMD:R_0402_1005Metric
- removed SW1: SW_Push, Button_Switch_SMD:SW_Push_1P1T_NO_Vertical_Wuerth_434133025816
- added J5: ~{FLASH}, Connector_PinSocket_2.54mm:PinSocket_1x02_P2.54mm_Vertical, F.Cu at (91.5, 76.0)
- added R22: 33, Capacitor_SMD:C_0603_1608Metric, F.Cu at (144.0, 88.7)
- added R23: 47, Capacitor_SMD:C_0603_1608Metric, F.Cu at (140.8, 86.5)
- added R24: 47, Capacitor_SMD:C_0603_1608Metric, F.Cu at (140.8, 88.8)
- added R25: 33, Capacitor_SMD:C_0603_1608Metric, F.Cu at (144.0, 91.2)
- added R26: 47, Capacitor_SMD:C_0603_1608Metric, F.Cu at (140.8, 91.2)
- C10, C6, C7, C9: value 4.7u -> 4.7uF
- R11, R15: value 560 -> 330; footprint Resistor_SMD:R_0402_1005Metric -> Capacitor_SMD:C_0603_1608Metric
- R12, R16: value 1100 -> 680; footprint Resistor_SMD:R_0402_1005Metric -> Capacitor_SMD:C_0603_1608Metric
- R14, R3: value 270 -> 150; footprint Resistor_SMD:R_0402_1005Metric -> Capacitor_SMD:C_0603_1608Metric
- R18: value 240 -> 150; footprint Resistor_SMD:R_0402_1005Metric -> Capacitor_SMD:C_0603_1608Metric
- R19: value 470 -> 330; footprint Resistor_SMD:R_0402_1005Metric -> Capacitor_SMD:C_0603_1608Metric
- R21: value 150 -> 33; footprint Resistor_SMD:R_0402_1005Metric -> Capacitor_SMD:C_0603_1608Metric
- SW2: footprint Button_Switch_SMD:SW_Push_1P1T_NO_Vertical_Wuerth_434133025816 -> Button_Switch_THT:SW_PUSH_6mm
- moved R21 9.36 mm to (144.0, 86.5), turned to 0 degrees
- moved SW2 8.27 mm to (118.0, 102.0), turned to -90 degrees
- moved R4 4.44 mm to (111.0, 108.5)
Connections:
- R21 pad 1: B -> Net-(R21-Pad1)
Routing:
- net +3V3: track 30.0 -> 115.1 mm, vias 0 -> 4
- net GND: track 140.7 -> 191.2 mm
- net LD0: track 66.7 -> 106.0 mm, vias 4 -> 0
- net R: track 12.5 -> 35.4 mm, vias 0 -> 1
- net LD7: track 68.0 -> 50.2 mm
- net LD3: track 70.9 -> 88.3 mm
- net G: track 11.9 -> 29.0 mm, vias 0 -> 1
- net B: track 10.7 -> 23.6 mm, vias 0 -> 1
- net LD6: track 63.4 -> 53.3 mm, vias 4 -> 2
- net /RUN: track 14.5 -> 23.9 mm, vias 0 -> 2
- net Net-(R4-Pad1): track 5.69 -> 15.0 mm
- net LD5: track 62.4 -> 56.2 mm
- net COL_G2: track 35.3 -> 39.8 mm
- net COL_G1: track 31.1 -> 33.5 mm
- net /~{USB_BOOT}: track 8.47 -> 6.17 mm
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Other:
- board text added: "jlcjlcjlcjlc"
- board text removed: "BOOTSEL"
