File: pcb/pico2-vga-adapter/pico2-vga-adapter.kicad_sch (KiCad schematic)
At the start: 71 parts, among them J1 USB_B_Micro, J2 VGA, J3 CONN, J4 SM03B-SRSS-TB, J5 Conn_01x08_Pin, J6 UART, Q1 BSS138, Q10 BSS138, Q2 BSS138, Q3 BSS138, Q4 BSS138, Q5 BSS138, Q6 BSS138, Q7 BSS138, Q8 BSS138, Q9 BSS138, SW1 SW_Push, SW2 SW_Push, U1 RP2350_60QFN, U2 NCP1117-3.3_SOT223, U3 W25Q128JVS, Y1 ABM8-272-T3

Commit message: Routing
Parts:
- removed Q1, Q10, Q2, Q3, Q4, Q5, Q6, Q7, Q8, Q9: BSS138, Package_TO_SOT_SMD:SOT-23, symbol Transistor_FET:BSS138
- removed RN1, RN2, RN3, RN4, RN5: 10k, Resistor_SMD:R_Array_Convex_4x0603, symbol Device:R_Pack04_Split
- added U4: SN74CBTD3861PWR, Package_SO:TSSOP-24_4.4x7.8mm_P0.65mm, symbol vera-module-rev4-rescue:74CBTLV3861-74xx
Connections:
- net +5V: now also U4.24 (VCC)
- net D0: now also U4.22 (B1)
- net D1: now also U4.21 (B2)
- net D2: now also U4.20 (B3)
- net D3: now also U4.19 (B4)
- net D4: now also U4.18 (B5)
- net D5: now also U4.17 (B6)
- net D6: now also U4.16 (B7)
- net D7: now also U4.15 (B8)
- net GND: now also U4.12 (GND), U4.23 (OE)
- net LATCH: now also U4.14 (B9)
- net LD0: now also U4.2 (A1)
- net LD1: now also U4.3 (A2)
- net LD2: now also U4.4 (A3)
- net LD3: now also U4.5 (A4)
- net LD4: now also U4.6 (A5)
- net LD5: now also U4.7 (A6)
- net LD6: now also U4.8 (A7)
- net LD7: now also U4.9 (A8)
- net L_LATCH: now also U4.10 (A9)
- net L_RX: now also U4.11 (A10)
- net TX: now also U4.13 (B10)

Commit message: Adding components
Parts:
- removed J5: Conn_01x08_Pin, symbol Connector:Conn_01x08_Pin
- BZ1: footprint (none) -> Buzzer_Beeper:Buzzer_15x7.5RM7.6
- C1, C19, C5: LCSC (none) -> C15850
- C11, C12, C13, C14, C15, C16, C17, C18, C2, C8: LCSC (none) -> C307331
- C3, C4: LCSC (none) -> C1548
- J1: LCSC (none) -> C428495
- L1: LCSC (none) -> C27999766
- R1: now not fitted
- R11, R12, R13, R14, R15, R16, R17, R18, R19, R21, R3: footprint (none) -> Resistor_SMD:R_0402_1005Metric
- R2, R4, R6: LCSC (none) -> C11702
- U1: LCSC (none) -> C42411118
- U2: LCSC (none) -> C6186
- U3: LCSC (none) -> C97521
- Y1: LCSC (none) -> C20625731
Connections:
- net GPIO22: no longer names the net of U1.34 (GPIO22)
- net GPIO23: no longer names the net of U1.35 (GPIO23)
- net GPIO24: no longer names the net of U1.36 (GPIO24)
- net GPIO25: no longer names the net of U1.37 (GPIO25)
- net GPIO26_ADC0: no longer names the net of U1.40 (GPIO26_ADC0)
- net GPIO27_ADC1: no longer names the net of U1.41 (GPIO27_ADC1)
- net GPIO28_ADC2: no longer names the net of U1.42 (GPIO28_ADC2)
- net GPIO29_ADC3: no longer names the net of U1.43 (GPIO29_ADC3)
- no-connect marks 7 -> 15

Commit message: Finalizing adapter design
Parts:
- removed R13, R17: 150, Resistor_SMD:R_0402_1005Metric, symbol Device:R
- removed SW1: SW_Push, Button_Switch_SMD:SW_Push_1P1T_NO_Vertical_Wuerth_434133025816, symbol Switch:SW_Push
- added J5: ~{FLASH}, Connector_PinSocket_2.54mm:PinSocket_1x02_P2.54mm_Vertical, symbol Connector:Conn_01x02_Pin
- added R22, R25: 33, Capacitor_SMD:C_0603_1608Metric, symbol Device:R
- added R23, R24, R26: 47, Capacitor_SMD:C_0603_1608Metric, symbol Device:R
- C10, C6, C7, C9: value 4.7u -> 4.7uF; LCSC (none) -> C1523
- J4: now not fitted
- R10: LCSC (none) -> C17168
- R11, R15: value 560 -> 330; footprint Resistor_SMD:R_0402_1005Metric -> Capacitor_SMD:C_0603_1608Metric; LCSC (none) -> C23138
- R12, R16: value 1100 -> 680; footprint Resistor_SMD:R_0402_1005Metric -> Capacitor_SMD:C_0603_1608Metric; LCSC (none) -> C23228
- R14, R3: value 270 -> 150; footprint Resistor_SMD:R_0402_1005Metric -> Capacitor_SMD:C_0603_1608Metric; LCSC (none) -> C22808
- R18: value 240 -> 150; footprint Resistor_SMD:R_0402_1005Metric -> Capacitor_SMD:C_0603_1608Metric; LCSC (none) -> C22808
- R19: value 470 -> 330; footprint Resistor_SMD:R_0402_1005Metric -> Capacitor_SMD:C_0603_1608Metric; LCSC (none) -> C23138
- R21: value 150 -> 33; footprint Resistor_SMD:R_0402_1005Metric -> Capacitor_SMD:C_0603_1608Metric; LCSC (none) -> C23140
- R5: LCSC (none) -> C25105
- R7, R8: LCSC (none) -> C25100
- SW2: footprint Button_Switch_SMD:SW_Push_1P1T_NO_Vertical_Wuerth_434133025816 -> Button_Switch_THT:SW_PUSH_6mm
- U4: LCSC (none) -> C2655473
Connections:
- net B: now also R23.1; no longer R21.1
- net G: now also R24.1
- net GND: now also J5.2 (Pin_2), R22.2, R25.2
- net R: now also R26.1
- net ~{USB_BOOT}: now also J5.1 (Pin_1)
- new net: R22.1, R24.2
- new net: R21.1, R23.2
- new net: R25.1, R26.2
Other:
- title: RP2350A QFN-60 Minimal Design Example -> PICO2-VGA-ADAPTER
- moved on the sheet: R14, R15, R16, R18, R19
